File: UWB_module.kicad_pcb (KiCad board)
At the start: 2 copper layers, 45 x 45 mm, 48 parts, among them J1 Conn_01x04_Female, J2 Conn_01x04_Male, J3 USB_B_Micro, J4 Conn_01x04_Male, U1 AZ1117-3.3, U3 STM32F103C8Tx, Y1 8.000M, Y2 32.768K

Commit message: Complete initial schematic and layout
Parts:
- moved C2 9.61 mm to (73.3, 77.5)
- moved D1 9.61 mm to (69.3, 77.2)
- moved C1 9.61 mm to (71.4, 77.4)
- moved C3 9.61 mm to (75.0, 77.5)
- moved Q1 9.61 mm to (69.5, 84.4)
- moved R19 5.72 mm to (67.4, 77.5), turned to 90 degrees
- moved D5 3.00 mm to (81.5, 75.0)
- moved D4 1.60 mm to (81.5, 69.5)
- moved D3 0.50 mm to (81.5, 64.3)
- moved D6 0.32 mm to (82.3, 84.3)
- moved C5 0.22 mm to (85.2, 90.3)
- moved C6 0.22 mm to (87.4, 90.3)
- moved U1 0.22 mm to (86.3, 84.1)
Connections:
- net /CAN_RX renamed Net-(U3-Pad45)
- net /CAN_TX renamed Net-(U3-Pad46)
- U3 pad 11: /TXLED -> Net-(U3-Pad11)
- U3 pad 14: /RXOKLED -> Net-(U3-Pad14)
- U3 pad 20: /RXLED -> Net-(U3-Pad20)
- U3 pad 38: Net-(U3-Pad38) -> /RXOKLED
- U3 pad 40: Net-(U3-Pad40) -> /RXLED
- U3 pad 41: Net-(U3-Pad41) -> /TXLED
Routing:
- net /USART2_RX: track 0.00 -> 29.3 mm
- net /USART2_TX: track 0.00 -> 26.4 mm
- net +3V3: track 191.5 -> 177.3 mm, vias 10 -> 9
- net +5V: track 47.5 -> 35.0 mm, vias 4 -> 2
- net Net-(J1-Pad1): track 17.7 -> 11.0 mm, vias 1 -> 0
- net /RXOKLED: track 26.4 -> 33.0 mm
- net /BOOT0: track 2.08 -> 8.63 mm
- net GND: track 9.95 -> 13.5 mm, vias 15 -> 22
- net /RXLED: track 26.1 -> 29.5 mm
- net /SFDLED: track 27.7 -> 31.1 mm
- net /TXLED: track 25.4 -> 28.3 mm
- net Net-(D5-Pad2): track 14.5 -> 17.4 mm
- net /USART1_RX: track 68.0 -> 66.3 mm
- net /USART1_TX: track 68.4 -> 66.9 mm
- net Net-(D4-Pad2): track 10.3 -> 11.7 mm
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Other:
- board text added: "USB"
- board text removed: "CAN"

Commit message: Add most up-to-date PCB and STEP file
Parts:
- removed Q1: ~, Package_TO_SOT_SMD:SOT-23
- added D2: NSR0530, Diode_SMD:D_SOD-323, F.Cu at (69.2, 84.1)
- added D7: NSR0530, Diode_SMD:D_SOD-323, F.Cu at (69.2, 82.0)
- added G***: OSHW_Logo_5mm, Logos:OSHW_Logo_5mm, B.Cu at (66.6, 58.6)
- D3, D4, D5: value LED Green -> APT1608LVBC/D; footprint LED_SMD:LED_1206_3216Metric -> LED_SMD:LED_0603_1608Metric
- D6: value MBR0520 -> NSR0530; footprint Diode_SMD:D_SOD-123 -> Diode_SMD:D_SOD-323
- moved D6 0.60 mm to (82.3, 83.8)
- moved R18 0.30 mm to (63.7, 91.4)
- moved D4 0.10 mm to (81.5, 69.6)
- moved D5 0.10 mm to (81.5, 74.9)
Connections:
- J3 pad 1: +5V -> VBUS
- R18 pad 1: +3V3 -> /USB_PULLUP
- U3 pad 42: Net-(U3-Pad42) -> /USB_PULLUP
Routing:
- net +5V: track 35.0 -> 10.1 mm, vias 2 -> 0
- net VBUS: track 0.00 -> 23.9 mm, vias 0 -> 2
- net /USB_PULLUP: track 0.00 -> 11.6 mm
- net /RXOKLED: track 33.0 -> 34.3 mm
- net /SFDLED: track 31.1 -> 32.0 mm
- net /RXLED: track 29.5 -> 30.3 mm
- net +3V3: track 177.3 -> 176.5 mm
- net GND: vias 22 -> 20
Other:
- board text removed: "H"
- board text removed: "L"
