File: UWB_module.sch (KiCad schematic (older format))
At the start: 48 parts, among them J1 Conn_01x04_Female, J2 Conn_01x04_Male, J3 USB_B_Micro, J4 Conn_01x04_Male, U1 AZ1117-3.3, U3 STM32F103C8Tx, Y1 8.000M, Y2 32.768K

Commit message: Complete initial schematic and layout
Connections:
- net RXLED: now also U3.40 (PB4); no longer U3.20 (PB2)
- net RXOKLED: now also U3.38 (PA15); no longer U3.14 (PA4)
- net TXLED: now also U3.41 (PB5); no longer U3.11 (PA1)
- net CAN_RX: no longer names the net of U3.45 (PB8)
- net CAN_TX: no longer names the net of U3.46 (PB9)
- no-connect marks 17 -> 18
Other:
- note added: "USB LED"
- note removed: "CAN OK"
Changed lines of the file:
@@
 $EndComp
 $Comp
-L power:GND #PWR03
+L power:GND #PWR?
 U 1 1 5D53BC0D
 P 3200 6200
-F 0 "#PWR03" H 3200 5950 50  0001 C CNN
+F 0 "#PWR?" H 3200 5950 50  0001 C CNN
 F 1 "GND" H 3205 6027 50  0000 C CNN
 F 2 "" H 3200 6200 50  0001 C CNN
@@
 	3200 3700 3300 3700
 $Comp
-L power:+3.3V #PWR02
+L power:+3.3V #PWR?
 U 1 1 5D53E827
 P 3200 3600
-F 0 "#PWR02" H 3200 3450 50  0001 C CNN
+F 0 "#PWR?" H 3200 3450 50  0001 C CNN
 F 1 "+3.3V" H 3215 3773 50  0000 C CNN
 F 2 "" H 3200 3600 50  0001 C CNN
@@
 NoConn ~ 2300 5000
 $Comp
-L power:GND #PWR01
+L power:GND #PWR?
 U 1 1 5D540233
 P 1800 4900
-F 0 "#PWR01" H 1800 4650 50  0001 C CNN
+F 0 "#PWR?" H 1800 4650 50  0001 C CNN
 F 1 "GND" H 1805 4727 50  0000 C CNN
 F 2 "" H 1800 4900 50  0001 C CNN
@@
 	5800 4900 5800 5550
 $Comp
-L power:GND #PWR05
+L power:GND #PWR?
 U 1 1 5D549C5B
 P 4300 6000
-F 0 "#PWR05" H 4300 5750 50  0001 C CNN
+F 0 "#PWR?" H 4300 5750 50  0001 C CNN
 F 1 "GND" H 4305 5827 50  0000 C CNN
 F 2 "" H 4300 6000 50  0001 C CNN
@@
 $EndComp
 $Comp
-L power:GND #PWR08
+L power:GND #PWR?
 U 1 1 5D557A7E
 P 5050 2250
-F 0 "#PWR08" H 5050 2000 50  0001 C CNN
+F 0 "#PWR?" H 5050 2000 50  0001 C CNN
 F 1 "GND" H 5055 2077 50  0000 C CNN
 F 2 "" H 5050 2250 50  0001 C CNN
@@
 $EndComp
 $Comp
-L power:+3.3V #PWR012
+L power:+3.3V #PWR?
 U 1 1 5D55ADE4
 P 6350 1600
-F 0 "#PWR012" H 6350 1450 50  0001 C CNN
+F 0 "#PWR?" H 6350 1450 50  0001 C CNN
 F 1 "+3.3V" H 6365 1773 50  0000 C CNN
 F 2 "" H 6350 1600 50  0001 C CNN
@@
 	5050 2200 5050 2250
 $Comp
-L power:+5V #PWR04
+L power:+5V #PWR?
 U 1 1 5D569E5B
 P 3250 1600
-F 0 "#PWR04" H 3250 1450 50  0001 C CNN
+F 0 "#PWR?" H 3250 1450 50  0001 C CNN
 F 1 "+5V" H 3265 1773 50  0000 C CNN
 F 2 "" H 3250 1600 50  0001 C CNN
@@
 $EndComp
 $Comp
-L power:GND #PWR013
+L power:GND #PWR?
 U 1 1 5D565D1A
 P 7600 3550
-F 0 "#PWR013" H 7600 3300 50  0001 C CNN
+F 0 "#PWR?" H 7600 3300 50  0001 C CNN
 F 1 "GND" H 7605 3377 50  0000 C CNN
 F 2 "" H 7600 3550 50  0001 C CNN
@@
 Connection ~ 8550 3350
 $Comp
-L power:+3.3V #PWR021
+L power:+3.3V #PWR?
 U 1 1 5D5793ED
 P 10200 2850
-F 0 "#PWR021" H 10200 2700 50  0001 C CNN
+F 0 "#PWR?" H 10200 2700 50  0001 C CNN
 F 1 "+3.3V" H 10215 3023 50  0000 C CNN
 F 2 "" H 10200 2850 50  0001 C CNN
@@
 	11700 3200 11850 3200
 $Comp
-L power:GND #PWR026
+L power:GND #PWR?
 U 1 1 5D5AB232
 P 11700 3300
-F 0 "#PWR026" H 11700 3050 50  0001 C CNN
+F 0 "#PWR?" H 11700 3050 50  0001 C CNN
 F 1 "GND" H 11705 3127 50  0000 C CNN
 F 2 "" H 11700 3300 50  0001 C CNN
@@
 $EndComp
 $Comp
-L power:GND #PWR022
+L power:GND #PWR?
 U 1 1 5D5ABC3C
 P 10500 6250
-F 0 "#PWR022" H 10500 6000 50  0001 C CNN
+F 0 "#PWR?" H 10500 6000 50  0001 C CNN
 F 1 "GND" H 10505 6077 50  0000 C CNN
 F 2 "" H 10500 6250 50  0001 C CNN
@@
 	7450 4350 7450 4550
 $Comp
-L power:GND #PWR014
+L power:GND #PWR?
 U 1 1 5D71EA8E
 P 7450 4550
-F 0 "#PWR014" H 7450 4300 50  0001 C CNN
+F 0 "#PWR?" H 7450 4300 50  0001 C CNN
 F 1 "GND" H 7455 4377 50  0000 C CNN
 F 2 "" H 7450 4550 50  0001 C CNN
@@
 	9500 9050 9500 8800
 $Comp
-L power:+3.3V #PWR015
+L power:+3.3V #PWR?
 U 1 1 5D7BFF67
 P 7800 10500
-F 0 "#PWR015" H 7800 10350 50  0001 C CNN
+F 0 "#PWR?" H 7800 10350 50  0001 C CNN
 F 1 "+3.3V" H 7815 10673 50  0000 C CNN
 F 2 "" H 7800 10500 50  0001 C CNN
@@
 $EndComp
 $Comp
-L power:GND #PWR018
+L power:GND #PWR?
 U 1 1 5D7C89C0
 P 9500 9450
-F 0 "#PWR018" H 9500 9200 50  0001 C CNN
+F 0 "#PWR?" H 9500 9200 50  0001 C CNN
 F 1 "GND" H 9505 9277 50  0000 C CNN
 F 2 "" H 9500 9450 50  0001 C CNN
@@
 Wire Wire Line
 	11200 5800 11000 5800
-Text Label 11200 4500 0    50   ~ 0
+Text Label 9200 4900 0    50   ~ 0
 TXLED
-Text Label 9200 4600 0    50   ~ 0
+Text Label 9200 4800 0    50   ~ 0
 RXLED
 Text Label 9200 4700 0    50   ~ 0
 SFDLED
-Text Label 11200 4800 0    50   ~ 0
+Text Label 11200 5900 0    50   ~ 0
 RXOKLED
 Wire Wire Line
-	11200 4500 11000 4500
-Wire Wire Line
 	11000 4600 11200 4600
 Wire Wire Line
 	11200 4700 11000 4700
-Wire Wire Line
-	11000 4800 11200 4800
 Text Label 11200 4900 0    50   ~ 0
 SPICLK
@@
 	10950 9050 10950 8800
 $Comp
-L power:+3.3V #PWR025
+L power:+3.3V #PWR?
 U 1 1 5D932949
 P 10950 8800
-F 0 "#PWR025" H 10950 8650 50  0001 C CNN
+F 0 "#PWR?" H 10950 8650 50  0001 C CNN
 F 1 "+3.3V" H 10965 8973 50  0000 C CNN
 F 2 "" H 10950 8800 50  0001 C CNN
@@
 $EndComp
 $Comp
-L power:GND #PWR024
+L power:GND #PWR?
 U 1 1 5D93D698
 P 10800 9450
-F 0 "#PWR024" H 10800 9200 50  0001 C CNN
+F 0 "#PWR?" H 10800 9200 50  0001 C CNN
 F 1 "GND" H 10805 9277 50  0000 C CNN
 F 2 "" H 10800 9450 50  0001 C CNN
@@
 Wire Wire Line
 	10700 9250 11050 9250
-Text Label 9200 5200 0    50   ~ 0
-CAN_RX
-Text Label 9200 5300 0    50   ~ 0
-CAN_TX
-Wire Wire Line
-	9200 5200 9700 5200
-Wire Wire Line
-	9200 5300 9700 5300
-NoConn ~ 9700 4800
-NoConn ~ 9700 4900
 NoConn ~ 9700 5000
 NoConn ~ 9700 5100
@@
 NoConn ~ 9700 5600
 NoConn ~ 9700 5700
-NoConn ~ 11000 5900
 NoConn ~ 11000 5200
 NoConn ~ 11000 4400
 NoConn ~ 9700 4000
 $Comp
-L power:GND #PWR017
+L power:GND #PWR?
 U 1 1 5DA77404
 P 8750 6450
-F 0 "#PWR017" H 8750 6200 50  0001 C CNN
+F 0 "#PWR?" H 8750 6200 50  0001 C CNN
 F 1 "GND" H 8755 6277 50  0000 C CNN
 F 2 "" H 8750 6450 50  0001 C CNN
@@
 	9600 5900 9700 5900
 Text Notes 8350 6250 0    50   ~ 0
-CAN OK
-$Comp
-L power:GND #PWR016
+USB LED
+$Comp
+L power:GND #PWR?
 U 1 1 5DB354D0
 P 8100 6550
-F 0 "#PWR016" H 8100 6300 50  0001 C CNN
+F 0 "#PWR?" H 8100 6300 50  0001 C CNN
 F 1 "GND" H 8105 6377 50  0000 C CNN
 F 2 "" H 8100 6550 50  0001 C CNN
@@
 	10000 1400 10000 1150
 $Comp
-L power:+5V #PWR020
+L power:+5V #PWR?
 U 1 1 5DC76E4E
 P 10000 1150
-F 0 "#PWR020" H 10000 1000 50  0001 C CNN
+F 0 "#PWR?" H 10000 1000 50  0001 C CNN
 F 1 "+5V" H 10015 1323 50  0000 C CNN
 F 2 "" H 10000 1150 50  0001 C CNN
@@
 $EndComp
 $Comp
-L power:GND #PWR019
+L power:GND #PWR?
 U 1 1 5DC84ABD
 P 9550 2150
-F 0 "#PWR019" H 9550 1900 50  0001 C CNN
+F 0 "#PWR?" H 9550 1900 50  0001 C CNN
 F 1 "GND" H 9555 1977 50  0000 C CNN
 F 2 "" H 9550 2150 50  0001 C CNN
@@
 $EndComp
 $Comp
-L power:+3.3V #PWR023
+L power:+3.3V #PWR?
 U 1 1 5DD97CE1
 P 10750 1150
-F 0 "#PWR023" H 10750 1000 50  0001 C CNN
+F 0 "#PWR?" H 10750 1000 50  0001 C CNN
 F 1 "+3.3V" H 10765 1323 50  0000 C CNN
 F 2 "" H 10750 1150 50  0001 C CNN
@@
 	5950 3700 5950 3800
 $Comp
-L power:GND #PWR027
+L power:GND #PWR?
 U 1 1 5D70E5EE
 P 5950 3800
-F 0 "#PWR027" H 5950 3550 50  0001 C CNN
+F 0 "#PWR?" H 5950 3550 50  0001 C CNN
 F 1 "GND" H 5955 3627 50  0000 C CNN
 F 2 "" H 5950 3800 50  0001 C CNN
@@
 $EndComp
 $Comp
-L power:GND #PWR029
+L power:GND #PWR?
 U 1 1 5D754D17
 P 11800 7650
-F 0 "#PWR029" H 11800 7400 50  0001 C CNN
+F 0 "#PWR?" H 11800 7400 50  0001 C CNN
 F 1 "GND" H 11805 7477 50  0000 C CNN
 F 2 "" H 11800 7650 50  0001 C CNN
@@
 $EndComp
 $Comp
-L power:GND #PWR030
+L power:GND #PWR?
 U 1 1 5D7A63BE
 P 12700 7650
-F 0 "#PWR030" H 12700 7400 50  0001 C CNN
+F 0 "#PWR?" H 12700 7400 50  0001 C CNN
 F 1 "GND" H 12705 7477 50  0000 C CNN
 F 2 "" H 12700 7650 50  0001 C CNN
@@
 $EndComp
 $Comp
-L power:GND #PWR031
+L power:GND #PWR?
 U 1 1 5D7B69C4
 P 13600 7650
-F 0 "#PWR031" H 13600 7400 50  0001 C CNN
+F 0 "#PWR?" H 13600 7400 50  0001 C CNN
 F 1 "GND" H 13605 7477 50  0000 C CNN
 F 2 "" H 13600 7650 50  0001 C CNN
@@
 $EndComp
 $Comp
-L power:GND #PWR032
+L power:GND #PWR?
 U 1 1 5D7C6DEC
 P 14500 7650
-F 0 "#PWR032" H 14500 7400 50  0001 C CNN
+F 0 "#PWR?" H 14500 7400 50  0001 C CNN
 F 1 "GND" H 14505 7477 50  0000 C CNN
 F 2 "" H 14500 7650 50  0001 C CNN
@@
 $EndComp
 $Comp
-L power:+3.3V #PWR0101
+L power:+3.3V #PWR?
 U 1 1 5D619D60
 P 9500 8800
-F 0 "#PWR0101" H 9500 8650 50  0001 C CNN
+F 0 "#PWR?" H 9500 8650 50  0001 C CNN
 F 1 "+3.3V" H 9515 8973 50  0000 C CNN
 F 2 "" H 9500 8800 50  0001 C CNN
@@
 USART2_RX
 Wire Wire Line
-	9200 4600 9700 4600
-Wire Wire Line
 	9200 4700 9700 4700
+NoConn ~ 9700 5200
+NoConn ~ 9700 5300
+Wire Wire Line
+	11000 5900 11200 5900
+Wire Wire Line
+	9200 4800 9700 4800
+NoConn ~ 11000 4500
+NoConn ~ 9700 4600
+Wire Wire Line
+	9200 4900 9700 4900
 $EndSCHEMATC

Commit message: Add most up-to-date PCB and STEP file
Parts:
- removed Q1: ~, Package_TO_SOT_SMD:SOT-23, symbol Device:Q_PMOS_GSD
- added D2, D7: NSR0530, Diode_SMD:D_SOD-323, symbol Diode:MBR0520
- D3, D4, D5: value LED Green -> APT1608LVBC/D; footprint LED_SMD:LED_1206_3216Metric -> LED_SMD:LED_0603_1608Metric
- D6: value MBR0520 -> NSR0530; footprint Diode_SMD:D_SOD-123 -> Diode_SMD:D_SOD-323
Connections:
- net +3V3: no longer R18.1
- net +5V: now also D2.1 (K), D7.1 (K); no longer J3.1 (VBUS)
- net USB_PULLUP: now reaches U3.42 (PB6)
- net USB_PULLUP: now also R18.1
- net at J1.1 (Pin_1): now also D2.2 (A)
- new net VBUS: D7.2 (A), J3.1 (VBUS)
- no-connect marks 18 -> 17
Other:
- moved on the sheet: R13
Changed lines of the file:
@@
 	3250 2150 3250 2200
 Wire Wire Line
-	3250 1600 3250 1750
+	3250 1200 3250 1350
 Wire Wire Line
 	5050 2050 5050 2200
@@
 L power:+5V #PWR?
 U 1 1 5D569E5B
-P 3250 1600
-F 0 "#PWR?" H 3250 1450 50  0001 C CNN
-F 1 "+5V" H 3265 1773 50  0000 C CNN
-F 2 "" H 3250 1600 50  0001 C CNN
-F 3 "" H 3250 1600 50  0001 C CNN
-	1    3250 1600
+P 3250 1200
+F 0 "#PWR?" H 3250 1050 50  0001 C CNN
+F 1 "+5V" H 3265 1373 50  0000 C CNN
+F 2 "" H 3250 1200 50  0001 C CNN
+F 3 "" H 3250 1200 50  0001 C CNN
+	1    3250 1200
 	1    0    0    -1
 $EndComp
@@
 	0    1    1    0
 $EndComp
-$Comp
-L Device:Q_PMOS_GSD Q1
-U 1 1 5D57C7A6
-P 2800 1850
-F 0 "Q1" V 3051 1850 50  0000 C CNN
-F 1 "~" V 3052 1850 50  0000 C CNN
-F 2 "Package_TO_SOT_SMD:SOT-23" H 3000 1950 50  0001 C CNN
-F 3 "~" H 2800 1850 50  0001 C CNN
-	1    2800 1850
-	0    -1   -1   0
-$EndComp
 Wire Wire Line
 	3000 1750 3250 1750
 Wire Wire Line
-	2600 1750 1950 1750
-Wire Wire Line
-	2800 2050 2800 2200
-Wire Wire Line
-	2800 2200 3250 2200
-Wire Wire Line
 	1950 2050 2250 2050
 Wire Wire Line
 	2250 2050 2250 2200
-Wire Wire Line
-	2250 2200 2800 2200
-Connection ~ 2800 2200
 $Comp
 L Device:C C1
@@
 P 6950 1950
 F 0 "D3" V 6989 1833 50  0000 R CNN
-F 1 "LED Green" V 6898 1833 50  0000 R CNN
-F 2 "LED_SMD:LED_1206_3216Metric" H 6950 1950 50  0001 C CNN
+F 1 "APT1608LVBC/D" V 6898 1833 50  0000 R CNN
+F 2 "LED_SMD:LED_0603_1608Metric" H 6950 1950 50  0001 C CNN
 F 3 "~" H 6950 1950 50  0001 C CNN
 	1    6950 1950
@@
 Wire Wire Line
 	10700 9250 11050 9250
-NoConn ~ 9700 5000
 NoConn ~ 9700 5100
 NoConn ~ 9700 5500
 NoConn ~ 9700 5600
 NoConn ~ 9700 5700
-NoConn ~ 11000 5200
 NoConn ~ 11000 4400
 NoConn ~ 9700 4000
@@
 	1    8750 6450
 	1    0    0    -1
-$EndComp
-$Comp
-L Device:LED D5
-U 1 1 5DA82A40
-P 8750 6200
-F 0 "D5" V 8789 6083 50  0000 R CNN
-F 1 "LED Green" V 8698 6083 50  0000 R CNN
-F 2 "LED_SMD:LED_1206_3216Metric" H 8750 6200 50  0001 C CNN
-F 3 "~" H 8750 6200 50  0001 C CNN
-	1    8750 6200
-	0    -1   -1   0
 $EndComp
 Wire Wire Line
@@
 Wire Wire Line
 	9600 5900 9700 5900
-Text Notes 8350 6250 0    50   ~ 0
+Text Notes 8350 6200 0    50   ~ 0
 USB LED
 $Comp
 L power:GND #PWR?
 U 1 1 5DB354D0
-P 8100 6550
-F 0 "#PWR?" H 8100 6300 50  0001 C CNN
-F 1 "GND" H 8105 6377 50  0000 C CNN
-F 2 "" H 8100 6550 50  0001 C CNN
-F 3 "" H 8100 6550 50  0001 C CNN
-	1    8100 6550
-	1    0    0    -1
-$EndComp
-$Comp
-L Device:LED D4
-U 1 1 5DB354D6
-P 8100 6300
-F 0 "D4" V 8139 6183 50  0000 R CNN
-F 1 "LED Green" V 8048 6183 50  0000 R CNN
-F 2 "LED_SMD:LED_1206_3216Metric" H 8100 6300 50  0001 C CNN
-F 3 "~" H 8100 6300 50  0001 C CNN
-	1    8100 6300
-	0    -1   -1   0
-$EndComp
-Wire Wire Line
-	8100 6450 8100 6550
-Text Notes 7700 6350 0    50   ~ 0
+P 7650 6450
+F 0 "#PWR?" H 7650 6200 50  0001 C CNN
+F 1 "GND" H 7655 6277 50  0000 C CNN
+F 2 "" H 7650 6450 50  0001 C CNN
+F 3 "" H 7650 6450 50  0001 C CNN
+	1    7650 6450
+	1    0    0    -1
+$EndComp
+Wire Wire Line
+	7650 6350 7650 6450
+Text Notes 7200 6350 0    50   ~ 0
 Ranging
 Wire Wire Line
-	9700 5800 9250 5800
+	9700 5800 8600 5800
 $Comp
 L Device:R_US R13
 U 1 1 5DB4DA74
-P 9100 5800
-F 0 "R13" V 8895 5800 50  0000 C CNN
-F 1 "330" V 8986 5800 50  0000 C CNN
-F 2 "Resistor_SMD:R_0603_1608Metric" V 9140 5790 50  0001 C CNN
-F 3 "~" H 9100 5800 50  0001 C CNN
-	1    9100 5800
+P 8450 5800
+F 0 "R13" V 8245 5800 50  0000 C CNN
+F 1 "330" V 8336 5800 50  0000 C CNN
+F 2 "Resistor_SMD:R_0603_1608Metric" V 8490 5790 50  0001 C CNN
+F 3 "~" H 8450 5800 50  0001 C CNN
+	1    8450 5800
 	0    1    1    0
 $EndComp
 Wire Wire Line
-	8950 5800 8100 5800
-Wire Wire Line
-	8100 5800 8100 6150
+	8300 5800 7650 5800
+Wire Wire Line
+	7650 5800 7650 6050
 $Comp
 L Connector:USB_B_Micro J3
@@
 F 3 "~" H 9700 1550 50  0001 C CNN
 	1    9550 1600
-	1    0    0    -1
-$EndComp
-Wire Wire Line
-	9850 1400 10000 1400
-Wire Wire Line
-	10000 1400 10000 1150
-$Comp
-L power:+5V #PWR?
-U 1 1 5DC76E4E
-P 10000 1150
-F 0 "#PWR?" H 10000 1000 50  0001 C CNN
-F 1 "+5V" H 10015 1323 50  0000 C CNN
-F 2 "" H 10000 1150 50  0001 C CNN
-F 3 "" H 10000 1150 50  0001 C CNN
-	1    10000 1150
 	1    0    0    -1
 $EndComp
@@
 	1    0    0    -1
 $EndComp
-$Comp
-L power:+3.3V #PWR?
-U 1 1 5DD97CE1
-P 10750 1150
-F 0 "#PWR?" H 10750 1000 50  0001 C CNN
-F 1 "+3.3V" H 10765 1323 50  0000 C CNN
-F 2 "" H 10750 1150 50  0001 C CNN
-F 3 "" H 10750 1150 50  0001 C CNN
-	1    10750 1150
-	1    0    0    -1
-$EndComp
 Wire Wire Line
 	10750 1450 10750 1600
@@
 P 5050 1150
 F 0 "D6" H 5050 934 50  0000 C CNN
-F 1 "MBR0520" H 5050 1025 50  0000 C CNN
-F 2 "Diode_SMD:D_SOD-123" H 5050 975 50  0001 C CNN
-F 3 "http://www.mccsemi.com/up_pdf/MBR0520~MBR0580(SOD123).pdf" H 5050 1150 50  0001 C CNN
+F 1 "NSR0530" H 5050 1025 50  0000 C CNN
+F 2 "Diode_SMD:D_SOD-323" H 5050 975 50  0001 C CNN
+F 3 "https://www.onsemi.com/pub/Collateral/NSR0530H-D.PDF" H 5050 1150 50  0001 C CNN
 	1    5050 1150
 	1    0    0    -1
@@
 Wire Wire Line
 	9200 4900 9700 4900
+Wire Wire Line
+	2250 2200 3250 2200
+$Comp
+L Device:LED D4
+U 1 1 5D62BA17
+P 7650 6200
+F 0 "D4" V 7689 6083 50  0000 R CNN
+F 1 "APT1608LVBC/D" V 7598 6083 50  0000 R CNN
+F 2 "LED_SMD:LED_0603_1608Metric" H 7650 6200 50  0001 C CNN
+F 3 "~" H 7650 6200 50  0001 C CNN
+	1    7650 6200
+	0    -1   -1   0
+$EndComp
+$Comp
+L Device:LED D5
+U 1 1 5D653111
+P 8750 6200
+F 0 "D5" V 8789 6083 50  0000 R CNN
+F 1 "APT1608LVBC/D" V 8698 6083 50  0000 R CNN
+F 2 "LED_SMD:LED_0603_1608Metric" H 8750 6200 50  0001 C CNN
+F 3 "~" H 8750 6200 50  0001 C CNN
+	1    8750 6200
+	0    -1   -1   0
+$EndComp
+Text Label 10900 950  0    50   ~ 0
+USB_PULLUP
+Wire Wire Line
+	10900 950  10750 950
+Wire Wire Line
+	10750 950  10750 1150
+Text Label 9200 5000 0    50   ~ 0
+USB_PULLUP
+NoConn ~ 11000 5200
+Wire Wire Line
+	9200 5000 9700 5000
+$Comp
+L power:VBUS #PWR?
+U 1 1 5D673BFD
+P 10000 1250
+F 0 "#PWR?" H 10000 1100 50  0001 C CNN
+F 1 "VBUS" H 10015 1423 50  0000 C CNN
+F 2 "" H 10000 1250 50  0001 C CNN
+F 3 "" H 10000 1250 50  0001 C CNN
+	1    10000 1250
+	1    0    0    -1
+$EndComp
+Wire Wire Line
+	10000 1250 10000 1400
+Wire Wire Line
+	9850 1400 10000 1400
+$Comp
+L Diode:MBR0520 D2
+U 1 1 5D6A637C
+P 2850 1750
+F 0 "D2" H 2850 1534 50  0000 C CNN
+F 1 "NSR0530" H 2850 1625 50  0000 C CNN
+F 2 "Diode_SMD:D_SOD-323" H 2850 1575 50  0001 C CNN
+F 3 "https://www.onsemi.com/pub/Collateral/NSR0530H-D.PDF" H 2850 1750 50  0001 C CNN
+	1    2850 1750
+	-1   0    0    1
+$EndComp
+$Comp
+L power:VBUS #PWR?
+U 1 1 5D664276
+P 2400 1200
+F 0 "#PWR?" H 2400 1050 50  0001 C CNN
+F 1 "VBUS" H 2415 1373 50  0000 C CNN
+F 2 "" H 2400 1200 50  0001 C CNN
+F 3 "" H 2400 1200 50  0001 C CNN
+	1    2400 1200
+	1    0    0    -1
+$EndComp
+Wire Wire Line
+	1950 1750 2700 1750
+$Comp
+L Diode:MBR0520 D7
+U 1 1 5D6F47E2
+P 2850 1350
+F 0 "D7" H 2850 1134 50  0000 C CNN
+F 1 "NSR0530" H 2850 1225 50  0000 C CNN
+F 2 "Diode_SMD:D_SOD-323" H 2850 1175 50  0001 C CNN
+F 3 "https://www.onsemi.com/pub/Collateral/NSR0530H-D.PDF" H 2850 1350 50  0001 C CNN
+	1    2850 1350
+	-1   0    0    1
+$EndComp
+Wire Wire Line
+	2400 1200 2400 1350
+Wire Wire Line
+	2400 1350 2700 1350
+Wire Wire Line
+	3000 1350 3250 1350
+Connection ~ 3250 1350
+Wire Wire Line
+	3250 1350 3250 1750
 $EndSCHEMATC
